File: input/input.kicad_pcb (KiCad board)
At the start: 2 copper layers, 54 parts, among them P1 CONN_02X04, P10 CONN_02X05, P11 CONN_02X05, P12 CONN_02X05, P13 CONN_02X05, P14 CONN_02X05, P15 CONN_02X05, P16 CONN_02X05, P17 CONN_02X05, P18 CONN_02X05, P2 CONN_01X03, P3 CONN_02X05, P4 CONN_02X05, P5 CONN_02X05, P6 CONN_02X05, P7 CONN_02X05, P8 CONN_02X05, P9 CONN_02X05, U1 CD4021, U10 CD4021, U11 CD4021, U12 CD4021, U13 CD4021, U14 CD4021, U15 CD4021, U16 CD4021, U2 CD4021, U3 CD4021, U4 CD4021, U5 CD4021, U6 CD4021, U7 CD4021, U8 CD4021, U9 CD4021

Commit message: Adapt avionica ports to 6 pins
Other:
- board text added: "Avionica Digital Input Expansion Board Rev.01 Copyright (C) 2017 Alvaro Polo"
- board text removed: "Avionica Digital Input Expansion Board Copyright (C) 2017 Alvaro Polo"
Changed lines of the file:
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@@
     (visible_elements 7FFFF7FF)
     (pcbplotparams
-      (layerselection 0x00030_80000001)
+      (layerselection 0x03030_80000001)
       (usegerberextensions false)
       (excludeedgelayer true)
@@
       (outputformat 1)
       (mirror false)
-      (drillshape 1)
+      (drillshape 0)
       (scaleselection 1)
-      (outputdirectory ""))
+      (outputdirectory gerber))
   )
   (net 0 "")
@@
   (gr_line (start 74.93 113.665) (end 85.725 113.665) (angle 90) (layer F.SilkS) (width 0.2))
   (gr_line (start 73.025 107.315) (end 73.025 135.255) (angle 90) (layer Margin) (width 0.2))
-  (gr_text "Avionica Digital Input \nExpansion Board\nCopyright (C) 2017 Alvaro Polo" (at 200.025 120.65 90) (layer F.SilkS)
+  (gr_text "Avionica Digital Input \nExpansion Board Rev.01\nCopyright (C) 2017 Alvaro Polo" (at 200.025 120.65 90) (layer F.SilkS)
     (effects (font (size 1 1) (thickness 0.15)) (justify left))
   )
