File: led-driver/led-driver.sch (KiCad schematic (older format))
At the start: 2 parts, among them P1 CONN_02X04, P2 CONN_01X02

Commit message: Adapt avionica ports to 6 pins
Parts:
- P1: footprint (none) -> avionica:idc-8p
- P2: value CONN_01X02 -> CONN_01X03; footprint (none) -> avionica:Jack_55_21; symbol CONN_01X02 -> CONN_01X03
Connections:
- net GND: now also P2.3 (P3)
Changed lines of the file:
@@
 $EndDescr
 $Comp
-L GND #PWR1
+L GND #PWR01
 U 1 1 586A85BC
 P 2050 2850
-F 0 "#PWR1" H 2050 2600 50  0001 C CNN
+F 0 "#PWR01" H 2050 2600 50  0001 C CNN
 F 1 "GND" H 2050 2700 50  0000 C CNN
 F 2 "" H 2050 2850 50  0000 C CNN
@@
 $EndComp
 $Comp
-L GND #PWR2
+L GND #PWR02
 U 1 1 586A85D7
 P 3400 3200
-F 0 "#PWR2" H 3400 2950 50  0001 C CNN
+F 0 "#PWR02" H 3400 2950 50  0001 C CNN
 F 1 "GND" H 3400 3050 50  0000 C CNN
 F 2 "" H 3400 3200 50  0000 C CNN
@@
 	2800 3000 2550 3000
 $Comp
-L CONN_01X02 P2
+L CONN_01X03 P2
 U 1 1 586C7B37
-P 7850 3600
-F 0 "P2" H 7850 3750 50  0000 C CNN
-F 1 "CONN_01X02" V 7950 3600 50  0000 C CNN
-F 2 "" H 7850 3600 50  0000 C CNN
-F 3 "" H 7850 3600 50  0000 C CNN
-	1    7850 3600
+P 7850 3650
+F 0 "P2" H 7850 3850 50  0000 C CNN
+F 1 "CONN_01X03" V 7950 3650 50  0000 C CNN
+F 2 "avionica:Jack_55_21" H 7850 3650 50  0001 C CNN
+F 3 "" H 7850 3650 50  0000 C CNN
+	1    7850 3650
 	-1   0    0    -1
 $EndComp
 $Comp
-L VCC #PWR3
+L VCC #PWR03
 U 1 1 586C8582
 P 8200 3400
-F 0 "#PWR3" H 8200 3250 50  0001 C CNN
+F 0 "#PWR03" H 8200 3250 50  0001 C CNN
 F 1 "VCC" H 8200 3550 50  0000 C CNN
 F 2 "" H 8200 3400 50  0000 C CNN
@@
 $EndComp
 $Comp
-L GND #PWR4
+L GND #PWR04
 U 1 1 586C8943
 P 8200 3850
-F 0 "#PWR4" H 8200 3600 50  0001 C CNN
+F 0 "#PWR04" H 8200 3600 50  0001 C CNN
 F 1 "GND" H 8200 3700 50  0000 C CNN
 F 2 "" H 8200 3850 50  0000 C CNN
@@
 	8200 3650 8200 3850
 $Comp
-L PWR_FLAG #FLG1
+L PWR_FLAG #FLG05
 U 1 1 586C90D6
 P 8550 3400
-F 0 "#FLG1" H 8550 3495 50  0001 C CNN
+F 0 "#FLG05" H 8550 3495 50  0001 C CNN
 F 1 "PWR_FLAG" H 8550 3580 50  0000 C CNN
 F 2 "" H 8550 3400 50  0000 C CNN
@@
 $EndComp
 $Comp
-L PWR_FLAG #FLG2
+L PWR_FLAG #FLG06
 U 1 1 586C915A
 P 8550 3850
-F 0 "#FLG2" H 8550 3945 50  0001 C CNN
+F 0 "#FLG06" H 8550 3945 50  0001 C CNN
 F 1 "PWR_FLAG" H 8550 4030 50  0000 C CNN
 F 2 "" H 8550 3850 50  0000 C CNN
@@
 F 0 "P1" H 3050 3100 50  0000 C CNN
 F 1 "CONN_02X04" H 3050 2600 50  0001 C CNN
-F 2 "" H 3050 1650 50  0000 C CNN
+F 2 "avionica:idc-8p" H 3050 1650 50  0001 C CNN
 F 3 "" H 3050 1650 50  0000 C CNN
 	1    3050 2850
 	1    0    0    -1
 $EndComp
+Wire Wire Line
+	8050 3750 8200 3750
+Connection ~ 8200 3750
 $EndSCHEMATC
