File: led-driver/line.sch (KiCad schematic (older format))
At the start: 8 parts, among them P3 CONN_02X08, P4 CONN_02X08, U1 MAX7219, U2 MAX7219

Commit message: Adapt avionica ports to 6 pins
Parts:
- C1, C2: footprint (none) -> Capacitors_ThroughHole:C_Disc_D3.0mm_W2.0mm_P2.50mm
- P3, P4: footprint (none) -> avionica:idc-16p
- R1, R2: footprint (none) -> Discret:R3
- U1, U2: footprint (none) -> Housings_DIP:DIP-24_W7.62mm
Changed lines of the file:
@@
 AR Path="/58767CCF/587644BB" Ref="U5"  Part="1"
 AR Path="/58768830/587644BB" Ref="U7"  Part="1"
-F 0 "U7" H 4100 4400 60  0000 C CNN
+F 0 "U1" H 4100 4400 60  0000 C CNN
 F 1 "MAX7219" V 4350 3700 60  0000 C CNN
-F 2 "" H 4350 2800 60  0001 C CNN
+F 2 "Housings_DIP:DIP-24_W7.62mm" H 4350 2800 60  0001 C CNN
 F 3 "" H 4350 2800 60  0001 C CNN
 	1    4350 3500
@@
 AR Path="/58767CCF/587644C2" Ref="U6"  Part="1"
 AR Path="/58768830/587644C2" Ref="U8"  Part="1"
-F 0 "U8" H 6300 4400 60  0000 C CNN
+F 0 "U2" H 6300 4400 60  0000 C CNN
 F 1 "MAX7219" V 6550 3700 60  0000 C CNN
-F 2 "" H 6550 2800 60  0001 C CNN
+F 2 "Housings_DIP:DIP-24_W7.62mm" H 6550 2800 60  0001 C CNN
 F 3 "" H 6550 2800 60  0001 C CNN
 	1    6550 3500
@@
 AR Path="/58767CCF/587644CC" Ref="P7"  Part="1"
 AR Path="/58768830/587644CC" Ref="P9"  Part="1"
-F 0 "P9" H 4350 5000 50  0000 C CNN
+F 0 "P3" H 4350 5000 50  0000 C CNN
 F 1 "CONN_02X08" V 4350 4550 50  0000 C CNN
-F 2 "" H 4350 3350 50  0000 C CNN
+F 2 "avionica:idc-16p" H 4350 3350 50  0001 C CNN
 F 3 "" H 4350 3350 50  0000 C CNN
 	1    4350 4550
@@
 AR Path="/58767CCF/587644DE" Ref="P8"  Part="1"
 AR Path="/58768830/587644DE" Ref="P10"  Part="1"
-F 0 "P10" H 6550 5000 50  0000 C CNN
+F 0 "P4" H 6550 5000 50  0000 C CNN
 F 1 "CONN_02X08" V 6550 4550 50  0000 C CNN
-F 2 "" H 6550 3350 50  0000 C CNN
+F 2 "avionica:idc-16p" H 6550 3350 50  0001 C CNN
 F 3 "" H 6550 3350 50  0000 C CNN
 	1    6550 4550
@@
 AR Path="/58767CCF/587644EB" Ref="R5"  Part="1"
 AR Path="/58768830/587644EB" Ref="R7"  Part="1"
-F 0 "R7" V 5230 2950 50  0000 C CNN
+F 0 "R1" V 5230 2950 50  0000 C CNN
 F 1 "R" V 5150 2950 50  0000 C CNN
-F 2 "" V 5080 2950 50  0000 C CNN
+F 2 "Discret:R3" V 5080 2950 50  0001 C CNN
 F 3 "" H 5150 2950 50  0000 C CNN
 	1    5150 2950
@@
 	5400 2850 4850 2850
 $Comp
-L VCC #PWR5
+L VCC #PWR07
 U 1 1 587644F6
 P 5400 2700
-AR Path="/58764210/587644F6" Ref="#PWR5"  Part="1"
-AR Path="/587670AE/587644F6" Ref="#PWR9"  Part="1"
-AR Path="/58767CCF/587644F6" Ref="#PWR13"  Part="1"
-AR Path="/58768830/587644F6" Ref="#PWR17"  Part="1"
-F 0 "#PWR17" H 5400 2550 50  0001 C CNN
+AR Path="/58764210/587644F6" Ref="#PWR07"  Part="1"
+AR Path="/587670AE/587644F6" Ref="#PWR011"  Part="1"
+AR Path="/58767CCF/587644F6" Ref="#PWR015"  Part="1"
+AR Path="/58768830/587644F6" Ref="#PWR019"  Part="1"
+F 0 "#PWR019" H 5400 2550 50  0001 C CNN
 F 1 "VCC" H 5400 2850 50  0000 C CNN
 F 2 "" H 5400 2700 50  0000 C CNN
@@
 AR Path="/58767CCF/587644FD" Ref="R6"  Part="1"
 AR Path="/58768830/587644FD" Ref="R8"  Part="1"
-F 0 "R8" V 7430 2950 50  0000 C CNN
+F 0 "R2" V 7430 2950 50  0000 C CNN
 F 1 "R" V 7350 2950 50  0000 C CNN
-F 2 "" V 7280 2950 50  0000 C CNN
+F 2 "Discret:R3" V 7280 2950 50  0001 C CNN
 F 3 "" H 7350 2950 50  0000 C CNN
 	1    7350 2950
@@
 	7200 2950 7050 2950
 $Comp
-L VCC #PWR7
+L VCC #PWR08
 U 1 1 58764509
 P 7600 2700
-AR Path="/58764210/58764509" Ref="#PWR7"  Part="1"
-AR Path="/587670AE/58764509" Ref="#PWR11"  Part="1"
-AR Path="/58767CCF/58764509" Ref="#PWR15"  Part="1"
-AR Path="/58768830/58764509" Ref="#PWR19"  Part="1"
-F 0 "#PWR19" H 7600 2550 50  0001 C CNN
+AR Path="/58764210/58764509" Ref="#PWR08"  Part="1"
+AR Path="/587670AE/58764509" Ref="#PWR012"  Part="1"
+AR Path="/58767CCF/58764509" Ref="#PWR016"  Part="1"
+AR Path="/58768830/58764509" Ref="#PWR020"  Part="1"
+F 0 "#PWR020" H 7600 2550 50  0001 C CNN
 F 1 "VCC" H 7600 2850 50  0000 C CNN
 F 2 "" H 7600 2700 50  0000 C CNN
@@
 DATA
 $Comp
-L GND #PWR6
+L GND #PWR09
 U 1 1 5876499A
 P 5400 3350
-AR Path="/58764210/5876499A" Ref="#PWR6"  Part="1"
-AR Path="/587670AE/5876499A" Ref="#PWR10"  Part="1"
-AR Path="/58767CCF/5876499A" Ref="#PWR14"  Part="1"
-AR Path="/58768830/5876499A" Ref="#PWR18"  Part="1"
-F 0 "#PWR18" H 5400 3100 50  0001 C CNN
+AR Path="/58764210/5876499A" Ref="#PWR09"  Part="1"
+AR Path="/587670AE/5876499A" Ref="#PWR013"  Part="1"
+AR Path="/58767CCF/5876499A" Ref="#PWR017"  Part="1"
+AR Path="/58768830/5876499A" Ref="#PWR021"  Part="1"
+F 0 "#PWR021" H 5400 3100 50  0001 C CNN
 F 1 "GND" H 5400 3200 50  0000 C CNN
 F 2 "" H 5400 3350 50  0000 C CNN
@@
 AR Path="/58767CCF/587649EA" Ref="C5"  Part="1"
 AR Path="/58768830/587649EA" Ref="C7"  Part="1"
-F 0 "C7" H 5410 3220 50  0000 L CNN
+F 0 "C1" H 5410 3220 50  0000 L CNN
 F 1 "C_Small" H 5410 3070 50  0001 L CNN
-F 2 "" H 5400 3150 50  0000 C CNN
+F 2 "Capacitors_ThroughHole:C_Disc_D3.0mm_W2.0mm_P2.50mm" H 5400 3150 50  0001 C CNN
 F 3 "" H 5400 3150 50  0000 C CNN
 	1    5400 3150
@@
 	5400 3350 5400 3250
 $Comp
-L GND #PWR8
+L GND #PWR010
 U 1 1 58764C11
 P 7600 3350
-AR Path="/58764210/58764C11" Ref="#PWR8"  Part="1"
-AR Path="/587670AE/58764C11" Ref="#PWR12"  Part="1"
-AR Path="/58767CCF/58764C11" Ref="#PWR16"  Part="1"
-AR Path="/58768830/58764C11" Ref="#PWR20"  Part="1"
-F 0 "#PWR20" H 7600 3100 50  0001 C CNN
+AR Path="/58764210/58764C11" Ref="#PWR010"  Part="1"
+AR Path="/587670AE/58764C11" Ref="#PWR014"  Part="1"
+AR Path="/58767CCF/58764C11" Ref="#PWR018"  Part="1"
+AR Path="/58768830/58764C11" Ref="#PWR022"  Part="1"
+F 0 "#PWR022" H 7600 3100 50  0001 C CNN
 F 1 "GND" H 7600 3200 50  0000 C CNN
 F 2 "" H 7600 3350 50  0000 C CNN
@@
 AR Path="/58767CCF/58764C17" Ref="C6"  Part="1"
 AR Path="/58768830/58764C17" Ref="C8"  Part="1"
-F 0 "C8" H 7610 3220 50  0000 L CNN
+F 0 "C2" H 7610 3220 50  0000 L CNN
 F 1 "C_Small" H 7610 3070 50  0001 L CNN
-F 2 "" H 7600 3150 50  0000 C CNN
+F 2 "Capacitors_ThroughHole:C_Disc_D3.0mm_W2.0mm_P2.50mm" H 7600 3150 50  0001 C CNN
 F 3 "" H 7600 3150 50  0000 C CNN
 	1    7600 3150
