File: kicad/keyboard/keyboard.sch (KiCad schematic (older format))
At the start: 2 parts, among them P1 CONN_02X04, P2 CONN_01X02

Commit message: Change the schematics of keypad controller to use an ATmega328
Parts:
- removed P1: CONN_02X04, symbol CONN_02X04
- removed P2: CONN_01X02, symbol CONN_01X02
- added C1, C2, C3: Capacitor, avionica:Disc_capacitor, symbol Capacitor
- added P1: CONN03, avionica:Jack_55_21, symbol CONN03
- added P2, P3, P4: CONN06, avionica:idc-6p, symbol CONN06
- added U1: atmega328, avionica:DIP-28, symbol atmega328
- added Y1: Crystal, avionica:Crystal, symbol Crystal
Connections:
- net labels removed: CLK, DATA.A, DATA.B, DATA.C, DATA.D, DAV.A, DAV.B, DAV.C, DAV.D, LATCH
- wire segments 38 -> 49
- no-connect marks 0 -> 4

Commit message: Add a MAX7219 to the keypad controller
Parts:
- added C2: 0.1uF, avionica:Disc_capacitor, symbol Capacitor
- added P5, P6: CONN08, avionica:idc-8p, symbol CONN08
- added R1: 10k, avionica:Axial_resistor, symbol Resistor
- added U2: MAX7219, avionica:DIP-24, symbol MAX7219
- C1: value Capacitor -> 0.1uF
- C3: renamed from C2; value Capacitor -> 22pF
- C4: renamed from C3; value Capacitor -> 22pF
Connections:
- wire segments 49 -> 76
- no-connect marks 4 -> 5

Commit message: Introduce a DAV signal in the Keypad Controller board
Connections:
- wire segments 76 -> 75
- no-connect marks 5 -> 4
Changed lines of the file:
@@
 EESchema Schematic File Version 2
-LIBS:keyboard-rescue
 LIBS:avionica
 LIBS:power
@@
 NoConn ~ 4900 3500
 NoConn ~ 4900 3600
-NoConn ~ 4900 3700
 $Comp
 L CONN06 P2
@@
 L GND #PWR03
 U 1 1 59F0800E
-P 6550 3200
-F 0 "#PWR03" H 6550 2950 50  0001 C CNN
-F 1 "GND" H 6550 3050 50  0000 C CNN
-F 2 "" H 6550 3200 60  0000 C CNN
-F 3 "" H 6550 3200 60  0000 C CNN
-	1    6550 3200
-	1    0    0    -1
-$EndComp
-Wire Wire Line
-	6550 3200 6550 3100
-Wire Wire Line
-	6500 3100 6600 3100
-Wire Wire Line
-	6500 3100 6500 3000
-Wire Wire Line
-	6600 3100 6600 3000
-Connection ~ 6550 3100
+P 6600 3200
+F 0 "#PWR03" H 6600 2950 50  0001 C CNN
+F 1 "GND" H 6600 3050 50  0000 C CNN
+F 2 "" H 6600 3200 60  0000 C CNN
+F 3 "" H 6600 3200 60  0000 C CNN
+	1    6600 3200
+	1    0    0    -1
+$EndComp
+Wire Wire Line
+	6600 3000 6600 3200
 $Comp
 L VCC #PWR04
@@
 	2750 2900 2950 2900
 Connection ~ 2750 3200
+Wire Wire Line
+	4900 3700 6500 3700
+Wire Wire Line
+	6500 3700 6500 3000
 $EndSCHEMATC

Commit message: Replace 2x6p IDC connectors by a single 12p in Keypad Controller board
Parts:
- removed P3, P4: CONN06, avionica:idc-6p, symbol CONN06
- added P3: CONN12, avionica:idc-12p, symbol CONN12
Connections:
- wire segments 75 -> 99
Changed lines of the file:
@@
 	3400 3100 3400 3200
 Wire Wire Line
-	3450 3600 3600 3600
-Wire Wire Line
-	3600 3700 3450 3700
-$Comp
-L CONN06 P3
-U 1 1 59F07B82
-P 3250 3850
-F 0 "P3" H 3250 4200 50  0000 C CNN
-F 1 "CONN06" V 3350 3850 50  0001 C CNN
-F 2 "avionica:idc-6p" H 3250 3850 60  0001 C CNN
-F 3 "" H 3250 3850 60  0000 C CNN
-	1    3250 3850
-	-1   0    0    -1
-$EndComp
-Wire Wire Line
-	3450 3800 3600 3800
-Wire Wire Line
-	3600 3900 3450 3900
-Wire Wire Line
-	3450 4000 3600 4000
-Wire Wire Line
-	3600 4100 3450 4100
-$Comp
-L CONN06 P4
-U 1 1 59F07C1B
-P 5250 3050
-F 0 "P4" H 5250 3400 50  0000 C CNN
-F 1 "CONN06" V 5350 3050 50  0001 C CNN
-F 2 "avionica:idc-6p" H 5250 3050 60  0001 C CNN
-F 3 "" H 5250 3050 60  0000 C CNN
-	1    5250 3050
-	1    0    0    -1
-$EndComp
+	1850 3600 3600 3600
+Wire Wire Line
+	1950 3700 3600 3700
+Wire Wire Line
+	2050 3800 3600 3800
+Wire Wire Line
+	2150 3900 3600 3900
+Wire Wire Line
+	2250 4000 3600 4000
+Wire Wire Line
+	2350 4100 3600 4100
 Wire Wire Line
 	4900 2800 5050 2800
 Wire Wire Line
-	5050 2900 4900 2900
-Wire Wire Line
-	4900 3000 5050 3000
-Wire Wire Line
-	5050 3100 4900 3100
-Wire Wire Line
-	4900 3200 5050 3200
-Wire Wire Line
-	5050 3300 4900 3300
+	4900 2900 5150 2900
+Wire Wire Line
+	4900 3000 5250 3000
+Wire Wire Line
+	4900 3100 5350 3100
+Wire Wire Line
+	4900 3200 5450 3200
+Wire Wire Line
+	4900 3300 5550 3300
 NoConn ~ 4900 3400
 NoConn ~ 4900 3500
@@
 Wire Wire Line
 	6500 3700 6500 3000
+$Comp
+L CONN12 P3
+U 1 1 59F9C051
+P 2400 1600
+F 0 "P3" H 2400 2250 50  0000 C CNN
+F 1 "CONN12" V 2500 1600 50  0001 C CNN
+F 2 "avionica:idc-12p" H 2400 1600 60  0001 C CNN
+F 3 "" H 2400 1600 60  0000 C CNN
+	1    2400 1600
+	0    -1   -1   0
+$EndComp
+Wire Wire Line
+	1850 3600 1850 1800
+Wire Wire Line
+	1950 3700 1950 1800
+Wire Wire Line
+	2050 1800 2050 3800
+Wire Wire Line
+	2150 3900 2150 1800
+Wire Wire Line
+	2250 1800 2250 4000
+Wire Wire Line
+	2350 4100 2350 1800
+Wire Wire Line
+	5050 2800 5050 2450
+Wire Wire Line
+	5050 2450 2450 2450
+Wire Wire Line
+	2450 2450 2450 1800
+Wire Wire Line
+	2550 1800 2550 2350
+Wire Wire Line
+	2550 2350 5150 2350
+Wire Wire Line
+	5150 2350 5150 2900
+Wire Wire Line
+	5250 3000 5250 2250
+Wire Wire Line
+	5250 2250 2650 2250
+Wire Wire Line
+	2650 2250 2650 1800
+Wire Wire Line
+	5350 3100 5350 2150
+Wire Wire Line
+	5350 2150 2750 2150
+Wire Wire Line
+	2750 2150 2750 1800
+Wire Wire Line
+	2850 1800 2850 2050
+Wire Wire Line
+	2850 2050 5450 2050
+Wire Wire Line
+	5450 2050 5450 3200
+Wire Wire Line
+	5550 3300 5550 1950
+Wire Wire Line
+	5550 1950 2950 1950
+Wire Wire Line
+	2950 1950 2950 1800
 $EndSCHEMATC

Commit message: Replace 2x8p IDC connectors by a single 16p in Keypad Controller board
Parts:
- removed P5, P6: CONN08, avionica:idc-8p, symbol CONN08
- added P4: CONN16, avionica:idc-16p, symbol CONN16
Connections:
- wire segments 99 -> 147
Changed lines of the file:
@@
 L MAX7219 U2
 U 1 1 59F0919B
-P 8200 3750
-F 0 "U2" H 8000 4650 60  0000 C CNN
-F 1 "MAX7219" H 8650 3250 60  0000 C CNN
-F 2 "avionica:DIP-24" H 8350 2950 60  0001 C CNN
-F 3 "" H 8350 2950 60  0001 C CNN
-	1    8200 3750
+P 8700 3750
+F 0 "U2" H 8500 4650 60  0000 C CNN
+F 1 "MAX7219" H 9150 3250 60  0000 C CNN
+F 2 "avionica:DIP-24" H 8850 2950 60  0001 C CNN
+F 3 "" H 8850 2950 60  0001 C CNN
+	1    8700 3750
 	1    0    0    -1
 $EndComp
@@
 	6400 3800 6400 3000
 Wire Wire Line
-	6950 3200 7700 3200
+	6950 3200 8200 3200
 Wire Wire Line
 	6950 4100 6950 3200
 Connection ~ 6100 4100
 Wire Wire Line
-	7700 3100 6850 3100
-Wire Wire Line
-	6850 3100 6850 3800
+	6850 3100 8200 3100
+Wire Wire Line
+	6850 3800 6850 3100
 Connection ~ 6400 3800
 Wire Wire Line
-	7700 3000 6750 3000
-Wire Wire Line
-	6750 3000 6750 3900
+	6750 3000 8200 3000
+Wire Wire Line
+	6750 3900 6750 3000
 Connection ~ 6300 3900
-NoConn ~ 8700 3000
+NoConn ~ 9200 3000
 $Comp
 L Resistor R1
 U 1 1 59F097DD
-P 8900 3100
-F 0 "R1" V 8900 3050 39  0000 L CNN
-F 1 "10k" V 9000 3050 50  0000 L CNN
-F 2 "avionica:Axial_resistor" H 8900 3100 60  0001 C CNN
-F 3 "" H 8900 3100 60  0000 C CNN
-	1    8900 3100
+P 9400 3100
+F 0 "R1" V 9400 3050 39  0000 L CNN
+F 1 "10k" V 9500 3050 50  0000 L CNN
+F 2 "avionica:Axial_resistor" H 9400 3100 60  0001 C CNN
+F 3 "" H 9400 3100 60  0000 C CNN
+	1    9400 3100
 	0    1    1    0
 $EndComp
@@
 L GND #PWR08
 U 1 1 59F09849
-P 9400 3200
-F 0 "#PWR08" H 9400 2950 50  0001 C CNN
-F 1 "GND" H 9400 3050 50  0000 C CNN
-F 2 "" H 9400 3200 60  0000 C CNN
-F 3 "" H 9400 3200 60  0000 C CNN
-	1    9400 3200
+P 9900 3200
+F 0 "#PWR08" H 9900 2950 50  0001 C CNN
+F 1 "GND" H 9900 3050 50  0000 C CNN
+F 2 "" H 9900 3200 60  0000 C CNN
+F 3 "" H 9900 3200 60  0000 C CNN
+	1    9900 3200
 	1    0    0    -1
 $EndComp
 Wire Wire Line
-	8700 3100 8800 3100
-$Comp
-L CONN08 P5
-U 1 1 59F09A83
-P 7300 3750
-F 0 "P5" H 7300 4200 50  0000 C CNN
-F 1 "CONN08" V 7400 3750 50  0001 C CNN
-F 2 "avionica:idc-8p" H 7300 3750 60  0001 C CNN
-F 3 "" H 7300 3750 60  0000 C CNN
-	1    7300 3750
-	-1   0    0    -1
-$EndComp
-$Comp
-L CONN08 P6
-U 1 1 59F09AD2
-P 9050 3750
-F 0 "P6" H 9050 4200 50  0000 C CNN
-F 1 "CONN08" V 9150 3750 50  0001 C CNN
-F 2 "avionica:idc-8p" H 9050 3750 60  0001 C CNN
-F 3 "" H 9050 3750 60  0000 C CNN
-	1    9050 3750
-	1    0    0    -1
-$EndComp
-Wire Wire Line
-	9000 3100 9400 3100
-Wire Wire Line
-	9400 3100 9400 3200
-Wire Wire Line
-	8850 3400 8700 3400
-Wire Wire Line
-	8700 3500 8850 3500
-Wire Wire Line
-	8850 3600 8700 3600
-Wire Wire Line
-	8850 3700 8700 3700
-Wire Wire Line
-	8850 3800 8700 3800
-Wire Wire Line
-	8850 3900 8700 3900
-Wire Wire Line
-	8850 4000 8700 4000
-Wire Wire Line
-	8850 4100 8700 4100
-Wire Wire Line
-	7500 3400 7700 3400
-Wire Wire Line
-	7700 3500 7500 3500
-Wire Wire Line
-	7500 3600 7700 3600
-Wire Wire Line
-	7700 3700 7500 3700
-Wire Wire Line
-	7500 3800 7700 3800
-Wire Wire Line
-	7700 3900 7500 3900
-Wire Wire Line
-	7500 4000 7700 4000
-Wire Wire Line
-	7700 4100 7500 4100
+	9200 3100 9300 3100
+Wire Wire Line
+	9500 3100 9900 3100
+Wire Wire Line
+	9900 3100 9900 3200
+Wire Wire Line
+	9200 3400 9450 3400
+Wire Wire Line
+	9200 3500 9550 3500
+Wire Wire Line
+	9200 3600 9650 3600
+Wire Wire Line
+	9200 3700 9750 3700
+Wire Wire Line
+	9200 3800 9850 3800
+Wire Wire Line
+	9200 3900 9950 3900
+Wire Wire Line
+	9200 4000 10050 4000
+Wire Wire Line
+	7300 3400 8200 3400
+Wire Wire Line
+	7400 3500 8200 3500
+Wire Wire Line
+	7500 3600 8200 3600
+Wire Wire Line
+	7600 3700 8200 3700
+Wire Wire Line
+	7700 3800 8200 3800
+Wire Wire Line
+	7800 3900 8200 3900
+Wire Wire Line
+	7900 4000 8200 4000
+Wire Wire Line
+	8200 4100 8000 4100
 $Comp
 L Capacitor C2
@@
 Wire Wire Line
 	2950 1950 2950 1800
+$Comp
+L CONN16 P4
+U 1 1 59FA0A7A
+P 8700 5300
+F 0 "P4" H 8700 6150 50  0000 C CNN
+F 1 "CONN16" V 8800 5300 50  0001 C CNN
+F 2 "avionica:idc-16p" H 8700 5300 60  0001 C CNN
+F 3 "" H 8700 5300 60  0000 C CNN
+	1    8700 5300
+	0    -1   1    0
+$EndComp
+Wire Wire Line
+	8000 4100 8000 4300
+Wire Wire Line
+	8000 4300 8650 4300
+Wire Wire Line
+	7900 4400 8550 4400
+Wire Wire Line
+	7900 4400 7900 4000
+Wire Wire Line
+	7800 3900 7800 4500
+Wire Wire Line
+	7800 4500 8450 4500
+Wire Wire Line
+	8650 4300 8650 5100
+Wire Wire Line
+	8550 4400 8550 5100
+Wire Wire Line
+	8450 4500 8450 5100
+Wire Wire Line
+	8350 5100 8350 4600
+Wire Wire Line
+	8350 4600 7700 4600
+Wire Wire Line
+	7700 4600 7700 3800
+Wire Wire Line
+	7600 3700 7600 4700
+Wire Wire Line
+	7600 4700 8250 4700
+Wire Wire Line
+	8250 4700 8250 5100
+Wire Wire Line
+	8150 5100 8150 4800
+Wire Wire Line
+	8150 4800 7500 4800
+Wire Wire Line
+	7500 4800 7500 3600
+Wire Wire Line
+	7400 3500 7400 4900
+Wire Wire Line
+	7400 4900 8050 4900
+Wire Wire Line
+	8050 4900 8050 5100
+Wire Wire Line
+	7950 5100 7950 5000
+Wire Wire Line
+	7950 5000 7300 5000
+Wire Wire Line
+	7300 5000 7300 3400
+Wire Wire Line
+	9450 3400 9450 4300
+Wire Wire Line
+	9450 4300 8750 4300
+Wire Wire Line
+	8750 4300 8750 5100
+Wire Wire Line
+	9550 3500 9550 4400
+Wire Wire Line
+	9550 4400 8850 4400
+Wire Wire Line
+	8850 4400 8850 5100
+Wire Wire Line
+	8950 5100 8950 4500
+Wire Wire Line
+	8950 4500 9650 4500
+Wire Wire Line
+	9650 4500 9650 3600
+Wire Wire Line
+	9750 3700 9750 4600
+Wire Wire Line
+	9750 4600 9050 4600
+Wire Wire Line
+	9050 4600 9050 5100
+Wire Wire Line
+	9150 5100 9150 4700
+Wire Wire Line
+	9150 4700 9850 4700
+Wire Wire Line
+	9850 4700 9850 3800
+Wire Wire Line
+	9250 5100 9250 4800
+Wire Wire Line
+	9250 4800 9950 4800
+Wire Wire Line
+	9950 4800 9950 3900
+Wire Wire Line
+	10050 4000 10050 4900
+Wire Wire Line
+	10050 4900 9350 4900
+Wire Wire Line
+	9350 4900 9350 5100
+Wire Wire Line
+	9450 5100 9450 5000
+Wire Wire Line
+	9450 5000 10150 5000
+Wire Wire Line
+	10150 5000 10150 4100
+Wire Wire Line
+	10150 4100 9200 4100
 $EndSCHEMATC

Commit message: Add a status LED to the Keypad Controller board
Parts:
- added D1: LED, avionica:LED-th, symbol LED
- added R2: 220, avionica:Axial_resistor, symbol Resistor
Connections:
- wire segments 147 -> 151
- no-connect marks 4 -> 3
Changed lines of the file:
@@
 NoConn ~ 4900 3400
 NoConn ~ 4900 3500
-NoConn ~ 4900 3600
 $Comp
 L CONN06 P2
@@
 U 1 1 59F097DD
 P 9400 3100
-F 0 "R1" V 9400 3050 39  0000 L CNN
-F 1 "10k" V 9500 3050 50  0000 L CNN
+F 0 "R1" V 9300 3100 39  0000 C CNN
+F 1 "10k" V 9400 3100 31  0000 C CNN
 F 2 "avionica:Axial_resistor" H 9400 3100 60  0001 C CNN
 F 3 "" H 9400 3100 60  0000 C CNN
@@
 Wire Wire Line
 	10150 4100 9200 4100
+$Comp
+L LED D1
+U 1 1 59FA2079
+P 5150 3600
+F 0 "D1" H 5100 3725 50  0000 L CNN
+F 1 "LED" H 5100 3600 50  0001 L CNN
+F 2 "avionica:LED-th" V 5150 3600 60  0001 C CNN
+F 3 "" V 5150 3600 60  0000 C CNN
+	1    5150 3600
+	-1   0    0    -1
+$EndComp
+$Comp
+L Resistor R2
+U 1 1 59FA20EB
+P 5450 3600
+F 0 "R2" V 5550 3550 39  0000 L CNN
+F 1 "220" V 5450 3600 31  0000 C CNN
+F 2 "avionica:Axial_resistor" H 5450 3600 60  0001 C CNN
+F 3 "" H 5450 3600 60  0000 C CNN
+	1    5450 3600
+	0    -1   -1   0
+$EndComp
+$Comp
+L GND #PWR09
+U 1 1 59FA212A
+P 5700 3550
+F 0 "#PWR09" H 5700 3300 50  0001 C CNN
+F 1 "GND" H 5700 3400 50  0000 C CNN
+F 2 "" H 5700 3550 60  0000 C CNN
+F 3 "" H 5700 3550 60  0000 C CNN
+	1    5700 3550
+	-1   0    0    1
+$EndComp
+Wire Wire Line
+	5250 3600 5350 3600
+Wire Wire Line
+	5550 3600 5700 3600
+Wire Wire Line
+	5700 3600 5700 3550
+Wire Wire Line
+	4900 3600 5050 3600
 $EndSCHEMATC
