File: kicad/keypad/keypad.kicad_pcb (KiCad board)
At the start: 2 copper layers, 18 parts, among them P1 CONN03, P2 CONN06, P3 CONN12, P4 CONN16, U1 atmega328, U2 MAX7219, Y1 Crystal

Commit message: Keypad controller Rev02: Update IDC connectors
Parts:
- C1, C2: value 0.1uF -> 100nF

Commit message: Fix wrong connection of ISET pin in Keypad Controller
Parts:
- C1, C2: value 100nF -> 0.1uF
- moved R1 10.2 mm to (179.7, 92.7), turned to 180 degrees
Connections:
- R1 pad 1: GND -> VCC
Routing:
- net VCC: track 80.2 -> 99.0 mm
Other:
- board text added: "Avionica Keypad Controller Board Rev02 Copyright (c) 2017 Alvaro Polo"
- board text removed: "Avionica Keypad Controller Board Rev01 Copyright (c) 2017 Alvaro Polo"
Changed lines of the file:
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@@
     (thickness 1.6)
     (drawings 9)
-    (tracks 287)
+    (tracks 292)
     (zones 0)
     (modules 18)
@@
   )
   (module avionica:Axial_resistor (layer F.Cu)
-    (at 169.545 92.71)
+    (at 179.705 92.71 180)
     (descr "Resistor, Axial_DIN0207 series, Axial, Horizontal, pin pitch=10.16mm, 0.25W = 1/4W, length*diameter=6.3*2.5mm^2, http://cdn-reichelt.de/documents/datenblatt/B400/1_4W%23YAG.pdf")
     (tags "Resistor Axial_DIN0207 series Axial Horizontal pin pitch 10.16mm 0.25W = 1/4W length 6.3mm diameter 2.5mm")
-    (fp_text reference R1 (at 10.795 2.54) (layer F.SilkS)
-      (effects (font (size 1 1) (thickness 0.15)))
-    )
-    (fp_text value 10k (at 5.08 0) (layer F.SilkS)
+    (fp_text reference R1 (at -1.905 1.27 180) (layer F.SilkS)
+      (effects (font (size 1 1) (thickness 0.15)))
+    )
+    (fp_text value 10k (at 5.08 0 180) (layer F.SilkS)
       (effects (font (size 1 1) (thickness 0.15)))
     )
@@
     (fp_line (start 11.25 1.6) (end 11.25 -1.6) (layer F.CrtYd) (width 0.05))
     (fp_line (start 11.25 -1.6) (end -1.05 -1.6) (layer F.CrtYd) (width 0.05))
-    (pad 1 thru_hole circle (at 0 0) (size 1.6 1.6) (drill 0.8) (layers *.Cu *.Mask)
-      (net 2 GND))
-    (pad 2 thru_hole oval (at 10.16 0) (size 1.6 1.6) (drill 0.8) (layers *.Cu *.Mask)
+    (pad 1 thru_hole circle (at 0 0 180) (size 1.6 1.6) (drill 0.8) (layers *.Cu *.Mask)
+      (net 1 VCC))
+    (pad 2 thru_hole oval (at 10.16 0 180) (size 1.6 1.6) (drill 0.8) (layers *.Cu *.Mask)
       (net 14 "Net-(R1-Pad2)"))
     (model ${KIPRJMOD}/../modules/packages3d/avionica.3dshapes/Axial_resistor.wrl
@@
       (effects (font (size 1 1) (thickness 0.15)))
     )
-    (fp_text value 100nF (at 0 0 180) (layer F.SilkS)
+    (fp_text value 0.1uF (at 0 0 180) (layer F.SilkS)
       (effects (font (size 0.7 0.7) (thickness 0.12)))
     )
@@
       (effects (font (size 1 1) (thickness 0.15)))
     )
-    (fp_text value 100nF (at 0 0 180) (layer F.SilkS)
+    (fp_text value 0.1uF (at 0 0 180) (layer F.SilkS)
       (effects (font (size 0.7 0.7) (thickness 0.12)))
     )
@@
     )
   )
-  (gr_text "Avionica Keypad Controller Board Rev01\nCopyright (c) 2017 Alvaro Polo\n" (at 162.56 100.965 90) (layer B.SilkS)
+  (gr_text "Avionica Keypad Controller Board Rev02\nCopyright (c) 2017 Alvaro Polo\n" (at 162.56 100.965 90) (layer B.SilkS)
     (effects (font (size 1 1) (thickness 0.2)) (justify left mirror))
   )
@@
   (gr_line (start 190 90) (end 190 140) (layer Margin) (width 0.2))
   (gr_line (start 140 90) (end 190 90) (layer Margin) (width 0.2))
+  (segment (start 177.8 92.71) (end 179.07 92.71) (width 0.25) (layer B.Cu) (net 1))
+  (segment (start 176.53 93.98) (end 177.8 92.71) (width 0.25) (layer B.Cu) (net 1))
+  (segment (start 176.53 94.615) (end 176.53 93.98) (width 0.25) (layer B.Cu) (net 1))
+  (segment (start 177.000001 108.420001) (end 176.53 107.95) (width 0.25) (layer B.Cu) (net 1))
+  (segment (start 176.53 107.95) (end 176.53 94.615) (width 0.25) (layer B.Cu) (net 1))
+  (segment (start 177.8 109.22) (end 177.000001 108.420001) (width 0.25) (layer B.Cu) (net 1))
   (segment (start 166.37 111.125) (end 167.64 111.125) (width 0.25) (layer F.Cu) (net 1))
   (segment (start 167.64 111.125) (end 168.275 110.49) (width 0.25) (layer F.Cu) (net 1))
@@
   (segment (start 163.195 99.695) (end 163.83 99.06) (width 0.25) (layer F.Cu) (net 13))
   (via (at 163.83 99.06) (size 0.6) (drill 0.4) (layers F.Cu B.Cu) (net 13))
-  (segment (start 179.705 92.71) (end 178.435 92.71) (width 0.25) (layer B.Cu) (net 14))
-  (segment (start 178.435 92.71) (end 175.895 95.25) (width 0.25) (layer B.Cu) (net 14))
-  (segment (start 175.895 95.25) (end 175.895 109.855) (width 0.25) (layer B.Cu) (net 14))
-  (segment (start 175.895 109.855) (end 177.8 111.76) (width 0.25) (layer B.Cu) (net 14))
+  (segment (start 177.8 111.76) (end 175.895 109.855) (width 0.25) (layer B.Cu) (net 14))
+  (segment (start 175.895 109.855) (end 175.895 99.06) (width 0.25) (layer B.Cu) (net 14))
+  (segment (start 175.895 99.06) (end 169.545 92.71) (width 0.25) (layer B.Cu) (net 14))
   (segment (start 149.225 130.81) (end 149.225 133.35) (width 0.25) (layer B.Cu) (net 15))
   (segment (start 149.225 133.35) (end 151.13 135.255) (width 0.25) (layer B.Cu) (net 15))
